Commit message: added table and paintgun

File: urdf/ur.urdf.xacro (robot description, xacro)
@@ -1,4 +1,4 @@
 <?xml version="1.0"?>
-<robot xmlns:xacro="http://wiki.ros.org/xacro" name="$(arg name)">
+<robot xmlns:xacro="http://wiki.ros.org/xacro" name="robot">
    <!-- robot name parameter -->
    <xacro:arg name="name" default="ur"/>
@@ -7,5 +7,5 @@
    <!-- possible 'ur_type' values: ur3, ur3e, ur5, ur5e, ur10, ur10e, ur16e, ur20, ur30 -->
    <!-- the default value should raise an error in case this was called without defining the type -->
-   <xacro:arg name="ur_type" default="ur5x"/>
+   <xacro:arg name="ur_type" default="ur10e"/>
    <!-- parameters -->
    <xacro:arg name="tf_prefix" default="" />
@@ -115,5 +115,6 @@
      trajectory_port="$(arg trajectory_port)"
      >
-     <origin xyz="0 0 0" rpy="0 0 0" />          <!-- position robot in the world -->
+     <origin xyz="0.0 0.0 0.0" rpy="0 0 0" />
+     <!-- <origin xyz="0.2 1.1471 0.88516" rpy="0 0 0" />  -->
    </xacro:ur_robot>
    <xacro:if value="$(arg sim_gazebo)">
@@ -138,3 +139,98 @@
     </gazebo>
   </xacro:if>
+  <link name="paintgun_base">
+    <visual>
+         <origin xyz="0.0 0.0455 0.06" rpy="0.0 0.0 0.0"/>
+         <geometry>
+           <mesh filename="package://ur_description/meshes/paintgun/paintgun_base.stl" scale="0.001 0.001 0.001"/>
+         </geometry>
+         <material name="blue">
+           <color rgba="0 0 1.0 1.0"/>
+         </material>
+       </visual>
+       <collision>
+         <origin xyz="0.0 0.0455 0.06" rpy="0.0 0.0 0.0"/>
+         <geometry>
+           <mesh filename="package://ur_description/meshes/paintgun/paintgun_base.stl" scale="0.001 0.001 0.001"/>
+         </geometry>
+       </collision>
+       <inertial>
+            <origin xyz="0.0 0.0 0.0" rpy="0.0 0.0 0.0"/>
+            <mass value="1.0"/>
+            <inertia ixx="1.0" ixy="0.0" ixz="0.0" iyy="1.0" iyz="0.0" izz="1.0"/>
+        </inertial>
+  </link>
+  <joint name="tool_to_paintgun_base" type="fixed">
+    <parent link="tool0"/>
+    <child link="paintgun_base"/>
+    <origin xyz="0.0 0.0 0.0" rpy="0.0 0.0 0.0"/>
+  </joint>
+  <link name="paintgun_handle">
+    <visual>
+    <origin xyz="0.0 0.0455 0.06" rpy="0.0 0.0 0.0"/>
+         <geometry>
+           <mesh filename="package://ur_description/meshes/paintgun/paintgun_handle.stl" scale="0.001 0.001 0.001"/>
+         </geometry>
+         <material name="blue">
+           <color rgba="0 0 1.0 1.0"/>
+         </material>
+       </visual>
+       <collision>
+    <origin xyz="0.0 0.0455 0.06" rpy="0.0 0.0 0.0"/>
+         <geometry>
+           <mesh filename="package://ur_description/meshes/paintgun/paintgun_handle.stl" scale="0.001 0.001 0.001"/>
+         </geometry>
+       </collision>
+       <inertial>
+            <origin xyz="0.0 0.0 0.0" rpy="0.0 0.0 0.0"/>
+            <mass value="1.0"/>
+            <inertia ixx="1.0" ixy="0.0" ixz="0.0" iyy="1.0" iyz="0.0" izz="1.0"/>
+        </inertial>
+  </link>
+  <joint name="paintgun_base_to_paintgun_handle" type="fixed">
+    <parent link="paintgun_base"/>
+    <child link="paintgun_handle"/>
+    <origin xyz="0.0 0.0 0.0" rpy="0.0 0.0 0.0"/>
+  </joint>
+  <link name="paintgun_marker">
+  </link>
+  <joint name="paintgun_handle_to_marker" type="fixed">
+    <parent link="paintgun_handle"/>
+    <child link="paintgun_marker"/>
+    <origin xyz="0.0 0.0485 0.04" rpy="0.0 0.0 0.0"/>
+  </joint>
+  <link name="paintgun_tcp">
+  </link>
+  <joint name="paintgun_handle_to_tcp" type="fixed">
+    <parent link="paintgun_handle"/>
+    <child link="paintgun_tcp"/>
+    <origin xyz="0.0 0.0295 0.170" rpy="0.0 0.0 0.0"/>
+  </joint>
+  <link name="ur_table">
+  <visual>
+    <origin xyz="1.19867 1.044 0.223" rpy="0.0 0.0 -1.57079632679"/>
+         <geometry>
+           <mesh filename="package://ur_description/meshes/table/ur_table.stl"/>
+         </geometry>
+         <material name="green">
+           <color rgba="0 1.0 0 1.0"/>
+         </material>
+       </visual>
+       <collision>
+    <origin xyz="1.19867 1.044 0.223" rpy="0.0 0.0 -1.57079632679"/>
+         <geometry>
+           <mesh filename="package://ur_description/meshes/table/ur_table.stl"/>
+         </geometry>
+       </collision>
+       <inertial>
+            <origin xyz="0.0 0.0 0.0" rpy="0.0 0.0 0.0"/>
+            <mass value="1.0"/>
+            <inertia ixx="1.0" ixy="0.0" ixz="0.0" iyy="1.0" iyz="0.0" izz="1.0"/>
+        </inertial>
+  </link>
+  <joint name="world_to_ur_table" type="fixed">
+    <parent link="world"/>
+    <child link="ur_table"/>
+    <origin xyz="-0.2 -1.1471 -0.88516" rpy="0.0 0.0 0.0"/>
+  </joint>
 </robot>

Commit message: changed initial position

File: urdf/ur.urdf.xacro (robot description, xacro)
@@ -72,5 +72,5 @@
      </link>
      <joint name="ground_plane_joint" type="fixed">
-       <origin xyz="0 0 -0.01" rpy="0 0 0"/>
+       <origin xyz="0 0 -0.88516" rpy="0 0 0"/>
        <parent link="world"/>
        <child link="ground_plane"/>

Commit message: changed init_position

File: urdf/ur.urdf.xacro (robot description, xacro)
@@ -164,5 +164,5 @@
     <parent link="tool0"/>
     <child link="paintgun_base"/>
-    <origin xyz="0.0 0.0 0.0" rpy="0.0 0.0 0.0"/>
+    <origin xyz="0.0 0.0 0.0" rpy="0.0 0.0 3.14159265359"/>
   </joint>
   <link name="paintgun_handle">

Commit message: adapted init rotation

File: urdf/ur.urdf.xacro (robot description, xacro)
@@ -115,5 +115,5 @@
      trajectory_port="$(arg trajectory_port)"
      >
-     <origin xyz="0.0 0.0 0.0" rpy="0 0 0" />
+     <origin xyz="0.0 0.0 0.0" rpy="0 0 -1.57079632679" />
      <!-- <origin xyz="0.2 1.1471 0.88516" rpy="0 0 0" />  -->
    </xacro:ur_robot>

Commit message: added aruco_base

File: urdf/ur.urdf.xacro (robot description, xacro)
@@ -200,4 +200,11 @@
     <origin xyz="0.0 0.0485 0.04" rpy="0.0 0.0 0.0"/>
   </joint>
+  <link name="aruco_base">
+  </link>
+  <joint name="world_to_aruco_base" type="fixed">
+    <parent link="world"/>
+    <child link="aruco_base"/>
+    <origin xyz="-0.05190672725439072 -0.8006927967071533 0.013048146851360798" rpy="-0.0316959 -0.028009 0.0328317"/>
+  </joint>
   <link name="paintgun_tcp">
   </link>
@@ -232,5 +239,5 @@
     <parent link="world"/>
     <child link="ur_table"/>
-    <origin xyz="-0.2 -1.1471 -0.88516" rpy="0.0 0.0 0.0"/>
+    <origin xyz="-0.135 -1.2121 -0.88516" rpy="0.0 0.0 0.0"/>
   </joint>
 </robot>

Commit message: corrected paintgun marker

File: urdf/ur.urdf.xacro (robot description, xacro)
@@ -193,10 +193,17 @@
     <origin xyz="0.0 0.0 0.0" rpy="0.0 0.0 0.0"/>
   </joint>
+  <link name="paintgun_marker_base">
+  </link>
+  <joint name="paintgun_handle_to_marker_base" type="fixed">
+    <parent link="paintgun_handle"/>
+    <child link="paintgun_marker_base"/>
+    <origin xyz="0.0 0.0485 0.04" rpy="0.0 0.0 0.0"/>
+  </joint>
   <link name="paintgun_marker">
   </link>
   <joint name="paintgun_handle_to_marker" type="fixed">
-    <parent link="paintgun_handle"/>
+    <parent link="paintgun_marker_base"/>
     <child link="paintgun_marker"/>
-    <origin xyz="0.0 0.0485 0.04" rpy="0.0 0.0 0.0"/>
+    <origin xyz="0.0 0.0 0.0" rpy="-1.57079632679 0.0 0.0"/>
   </joint>
   <link name="aruco_base">
